Commit message: miercoles14

File: src/dexarm_robot/urdf/simpledexarm.urdf (robot description, URDF)
Before this commit: robot DexArm_unofficial, 3 links, 2 joints
Links:
- link B_Fix: geometry collision mesh filename=file:./STL/00-B_Fix.stl scale=0.001 0.001 0.001; visual mesh filename=file:./STL/00-B_Fix.stl scale=0.001 0.001 0.001
- link B_Rot: geometry collision mesh filename=file:./STL/01-B_Rot.stl scale=0.001 0.001 0.001; visual mesh filename=file:./STL/01-B_Rot.stl scale=0.001 0.001 0.001
